File: Water Alarm/Water Alarm.kicad_pcb (KiCad board)
At the start: 2 copper layers, 8 parts, among them J1 Jack-DC, J2 Screw_Terminal_01x02, Q1 2N7000

Commit message: Added Water Alarm changes
Parts:
- moved G*** 5.79 mm to (151.7, 123.0)
Routing:
- net GND: track 0.00 -> 127.5 mm
- net VCC: track 0.00 -> 103.0 mm
- net /Gate: track 0.00 -> 51.0 mm
- net Net-(BZ1--): track 0.00 -> 32.1 mm
- added copper zone on B.Cu, net GND
Other:
- board outline added: 56.6 x 48.6 mm
