File: amplifier/amplifier.kicad_sch (KiCad schematic)
At the start: 13 parts, among them J1 INPUT, J2 OUTPUT, J3 POWER IN, Q1 TIP41, Q2 TIP42, U1 LM833

Commit message: Added amplifier
Other:
- moved on the sheet: U1C
Changed lines of the file:
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@@
 	(wire
 		(pts
-			(xy 54.61 156.21) (xy 54.61 161.29)
+			(xy 54.61 134.62) (xy 54.61 139.7)
 		)
 		(stroke
@@
 	(wire
 		(pts
-			(xy 54.61 176.53) (xy 54.61 184.15)
+			(xy 54.61 154.94) (xy 54.61 162.56)
 		)
 		(stroke
@@
 	(global_label "-12V"
 		(shape input)
-		(at 54.61 184.15 270)
+		(at 54.61 162.56 270)
 		(fields_autoplaced yes)
 		(effects
@@
 		)
 		(property "Intersheetrefs" "${INTERSHEET_REFS}"
-			(at 54.61 192.2152 90)
+			(at 54.61 170.6252 90)
 			(hide yes)
 			(show_name no)
@@
 	(global_label "+12V"
 		(shape input)
-		(at 54.61 156.21 90)
+		(at 54.61 134.62 90)
 		(fields_autoplaced yes)
 		(effects
@@
 		)
 		(property "Intersheetrefs" "${INTERSHEET_REFS}"
-			(at 54.61 148.1448 90)
+			(at 54.61 126.5548 90)
 			(hide yes)
 			(show_name no)
@@
 	(symbol
 		(lib_id "Amplifier_Operational:TL072")
-		(at 57.15 168.91 0)
+		(at 57.15 147.32 0)
 		(unit 3)
 		(body_style 1)
@@
 		(fields_autoplaced yes)
 		(property "Reference" "U1"
-			(at 55.88 167.6399 0)
+			(at 55.88 146.0499 0)
 			(show_name no)
 			(do_not_autoplace no)
@@
 		)
 		(property "Value" "LM833"
-			(at 55.88 170.1799 0)
+			(at 55.88 148.5899 0)
 			(show_name no)
 			(do_not_autoplace no)
@@
 		)
 		(property "Footprint" "Package_DIP:DIP-8_W7.62mm_LongPads"
-			(at 57.15 168.91 0)
+			(at 57.15 147.32 0)
 			(hide yes)
 			(show_name no)
@@
 		)
 		(property "Datasheet" "http://www.ti.com/lit/ds/symlink/tl071.pdf"
-			(at 57.15 168.91 0)
+			(at 57.15 147.32 0)
 			(hide yes)
 			(show_name no)
@@
 		)
 		(property "Description" "Dual Low-Noise JFET-Input Operational Amplifiers, DIP-8/SOIC-8"
-			(at 57.15 168.91 0)
-			(hide yes)
-			(show_name no)
+			(at 57.15 147.32 0)
+			(hide yes)
+			(show_name no)
